File: hardware/c6-carrier-rev-a/planter-c6-rev-a.kicad_sch (KiCad schematic)
At the start: 26 parts, among them J1 PROTECTED BATTERY, J2 MOISTURE PROBE, J3 WEACT 1.54 INCH, Q1 AO3401A, U1 Seeed XIAO ESP32-C6

Commit message: Reconcile C6 schematic with perfboard P1 (rev A-P1)
Annotate perfboard terminals, JP1 and PACK+/GND test pads; record bench
battery check. Connectivity unchanged; ERC clean. SVG re-exported.

Co-Authored-By: Claude Opus 5.5 <noreply@anthropic.com>
Other:
- note added: "J2: perfboard B06 VCC, B05 AOUT, B04 GND. J3 pins 1-8: perfboard B15 down to B08; WeAct B&W tested."
- note added: "P1 guide: 50 x 70mm perfboard, A-R / 01-24. JP1 = O01-O02 (letter O); TP1 PACK+ = K03; TP2 GND = K07. Battery-only check: display 3.81V / meter 3.83V. Air/water endpoints and WeAct 1.54-inch B&W refresh tested. Sleep current, protection specifications, USB charge behaviour and outdoor endurance remain unverified. Retain external 1S protection; never join B- to GND. U1/J1/J2/J3 footprints and PCB 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"
- note removed: "J2 keyed part TBD. C4 at U1; C5 at J2. J3 odd/even pinout from WeAct drawing; cable orientation TBD."
- note removed: "No on-carrier lithium protection or duplicate charger. Identify and insulate the external protection board. J1/J2/J3 and U1 footprints are intentionally unassigned pending exact parts and mechanical checks. Confirm actual display controller, cable ESD requirements, enclosure clearances and charging access. Before field use: polarity/continuity, ADC calibration, rail-off leakage, USB charging and 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"
- title: Planter XIAO ESP32-C6 carrier -> Planter XIAO ESP32-C6 carrier / perfboard P1
Changed lines of the file:
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@@
 (kicad_sch (version 20250114) (generator "planter_capture") (paper "A3")
-(title_block (title "Planter XIAO ESP32-C6 carrier") (date "2026-09-05") (rev "A") (comment 1 "External protected 1S pack; not fabrication-ready"))
+(title_block (title "Planter XIAO ESP32-C6 carrier / perfboard P1") (date "2026-09-09") (rev "A-P1") (comment 1 "Perfboard guide reconciled; not fabrication-ready"))
 (symbol (lib_id "Planter:Conn_01x02") (at 50.8 50.8 0) (unit 1) (in_bom yes) (on_board yes) (dnp no)
 (property "Reference" "J1" (at 50.8 43.18 0) (effects (font (size 1.27 1.27))))
@@
 (text "05  PROBE / FILTER" (at 213 127 0) (effects (font (size 2 2)) (justify left top)))
 (text "06  DISPLAY / LOCAL BYPASS" (at 327 127 0) (effects (font (size 2 2)) (justify left top)))
-(text "J2 keyed part TBD. C4 at U1; C5 at J2.\nJ3 odd/even pinout from WeAct drawing; cable orientation TBD." (at 213 202 0) (effects (font (size 1.5 1.5)) (justify left top)))
+(text "J2: perfboard B06 VCC, B05 AOUT, B04 GND.\nJ3 pins 1-8: perfboard B15 down to B08; WeAct B&W tested." (at 213 202 0) (effects (font (size 1.5 1.5)) (justify left top)))
 (text "07  TEST POINTS" (at 20 212 0) (effects (font (size 2 2)) (justify left top)))
 (text "PROTOTYPE CAPTURE - NOT A FABRICATION RELEASE" (at 20 243 0) (effects (font (size 2 2)) (justify left top)))
-(text "No on-carrier lithium protection or duplicate charger. Identify and insulate the external protection board.\nJ1/J2/J3 and U1 footprints are intentionally unassigned pending exact parts and mechanical checks.\nConfirm actual display controller, cable ESD requirements, enclosure clearances and charging access.\nBefore field use: polarity/continuity, ADC calibration, rail-off leakage, USB charging and 24-hour bench soak." (at 20 251 0) (effects (font (size 1.5 1.5)) (justify left top)))
+(text "P1 guide: 50 x 70mm perfboard, A-R / 01-24. JP1 = O01-O02 (letter O); TP1 PACK+ = K03; TP2 GND = K07.\nBattery-only check: display 3.81V / meter 3.83V. Air/water endpoints and WeAct 1.54-inch B&W refresh tested.\nSleep current, protection specifications, USB charge behaviour and outdoor endurance remain unverified.\nRetain external 1S protection; never join B- to GND. U1/J1/J2/J3 footprints and PCB layout remain pending." (at 20 251 0) (effects (font (size 1.5 1.5)) (justify left top)))
 (sheet_instances (path "/" (page "1"))))
